File: hardware/schematics/Sensorboard/SensorBee/SensorBee.kicad_sch (KiCad schematic)
At the start: 11 parts, among them J1 LiPo, J2 Sensor, U1 WEMOS_C3_mini, U2 HX711, U3 TP4056-42-ESOP8

Commit message: feat(sensorboard): INA226, Web-Dashboard, Memory-Bank + Schematics-Update
Sensorboard:
- INA226 Strom-/Leistungsmessung integriert (k0i05/esp_ina226 v1.2.7)
- elec-Topic (5s) über RS485 und HTTP-API
- Web-Dashboard (SPIFFS, /api/*, mDNS Womo-Sensor.local)
- Memory-Bank angelegt (projectbrief, techContext, systemPatterns, productContext, activeContext, progress)
- Claude Code Settings hinzugefügt (.claude/)

Hardware:
- SensorBee + Sensorboard KiCad-Schematics aktualisiert
- Exportierte PDF/SVG-Fab-Ausgaben hinzugefügt
- Auto-Saved-File entfernt

Sonstiges:
- Root CLAUDE.md hinzugefügt
- Router-WebUI und Website aktualisiert
- Ducato-Bild-Assets (sdcard/images) hinzugefügt

Co-Authored-By: Claude Sonnet 4.6 <noreply@anthropic.com>
Parts:
- added J3: USB_C_Receptacle_PowerOnly_6P, symbol Connector:USB_C_Receptacle_PowerOnly_6P
Connections:
- new net: J3.A12 (GND), J3.B12 (GND)
- new net: J3.A9 (VBUS), J3.B9 (VBUS)
Changed lines of the file:
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@@
+	)
+	(symbol
+		(lib_id "Connector:USB_C_Receptacle_PowerOnly_6P")
+		(at 181.61 85.09 0)
+		(unit 1)
+		(exclude_from_sim no)
+		(in_bom yes)
+		(on_board yes)
+		(dnp no)
+		(fields_autoplaced yes)
+		(property "Reference" "J3"
+			(at 181.61 67.31 0)
+			(effects
+				(font
+					(size 1.27 1.27)
+				)
+			)
+		)
+		(property "Value" "USB_C_Receptacle_PowerOnly_6P"
+			(at 181.61 69.85 0)
+			(effects
+				(font
+					(size 1.27 1.27)
+				)
+			)
+		)
+		(property "Footprint" ""
+			(at 185.42 82.55 0)
+			(effects
+				(font
+					(size 1.27 1.27)
+				)
+				(hide yes)
+			)
+		)
+		(property "Datasheet" "https://www.usb.org/sites/default/files/documents/usb_type-c.zip"
+			(at 181.61 85.09 0)
+			(effects
+				(font
+					(size 1.27 1.27)
+				)
+				(hide yes)
+			)
+		)
+		(property "Description" "USB Power-Only 6P Type-C Receptacle connector"
+			(at 181.61 85.09 0)
+			(effects
+				(font
+					(size 1.27 1.27)
+				)
+				(hide yes)
+			)
+		)
+		(pin "S1"
+		)
+		(pin "A12"
+		)
+		(pin "A9"
+		)
+		(pin "B12"
+		)
+		(pin "B9"
+		)
+		(pin "A5"
+		)
+		(pin "B5"
+		)
+		(instances
+			(project ""
+				(path "/9f8fd182-f53d-4129-ae8a-00de55493cce"
+					(reference "J3")
+					(unit 1)
+				)
+			)
+		)
 	)
 	(symbol
