File: hardware/schematics/ruuvitag_gas/ruuvitag_gas.kicad_sch (KiCad schematic)
At the start: 64 parts, among them P19 TP, P20 TP, P21 TP, P22 TP, P26 Ruuvi Connector, P5 RUUVI_BATTERY_CLIP, SW1 SW_PUSH, U1 nRF52832-QFAA, U2 DPS310XTSA1, U3 SHTC3, U4 LIS2DH12, Y1 32k, Y2 32M

Commit message: feat(hardware): ruuvitag_gas Phase 2a - HX711-Schaltplan umgesetzt
Rückbau TMP117/DPS310/LIS2DH12 samt SPI-/ACC-Netzen. HX711 (U2) mit
Load-Switch nach Option B: P-MOSFET High-Side (Q2) von VDD, N-MOSFET
Gate-Treiber (Q1) an HX711_EN -> nRF P0.03. Bridge/HX711 im Ruhezustand
stromlos, volle Ratiometrie.

- INA-Eingang: R5/R6 1k in Reihe, C6 100n differentiell, C2/C4 1n->GND (DNP)
- Entkopplung: C5 10u + C3 100n (AVDD), C15 100n (DVDD), C7 100n (VBG)
- Wägezellen-Pads J1-J4 (E+/E-/A+/A-), ext. Speise-Pads J5/J6 (DNP)
- SCK->P0.07, DOUT->P0.08 (nRF U1); SHTC3 = U4 auf Sensor_Humidity:SHTC3
- Y2->Y3: 32-MHz-Quarz auf Device:Crystal_GND24_Small
- Symbole/Footprints auf KiCad-Standardbibliotheken; alle 73 Bauteile mit FP
- ERC = 3 (alle erwartet: 2x pin_to_pin PWR_FLAG, 1x Antennen-Endpunkt)

Details und Bezeichner-Mapping: PHASE2_HX711.md §8. PCB (Phase 2b) offen.

Co-Authored-By: Claude Sonnet 5 <noreply@anthropic.com>
Claude-Session: https://claude.ai/code/session_01TiohMjQXZk3TSBS5rL6Eup
Parts:
- removed C12: 12p, RuuviTag:0402_CAP, symbol Device:C
- removed C17: 1u, RuuviTag:0402_CAP, symbol Device:C
- removed C18: 4u7, RuuviTag:0603_CAP, symbol Device:C
- removed P12, P2, P3: ~, RuuviTag:TEST_POINT_SMD_1MM, symbol Connector_Generic:Conn_01x01
- removed P6: ~, RuuviTag:FIDUCIAL_1MM, symbol Connector_Generic:Conn_01x01
- removed U1: nRF52832-QFAA, RuuviTag:QFN-48_6X6MM_BOTPAD, symbol nrf52832:nRF52832
- removed U2: DPS310XTSA1, RuuviTag:DPS310, symbol bmxx80:BMXX80
- removed U3: SHTC3, RuuviTag:DFN4_2X2MM_BOTPAD, symbol shtc3:SHTC3
- removed U4: LIS2DH12, RuuviTag:LGA12_2X2MM, symbol lis2dh12:LIS2Dx12
- removed U5: ~, RuuviTag:WSON6_NO_BOTPAD, symbol tmp117:TMP117
- removed Y2: 32M, RuuviTag:20X16MM_4PIN_CRYSTAL, symbol 4pin_crystal:4PIN_CRYSTAL
- added C15, C3, C6, C7: 100n, Capacitor_SMD:C_0402_1005Metric, symbol Device:C
- added C4: 1n, Capacitor_SMD:C_0402_1005Metric, symbol Device:C
- added C5: 10u, Capacitor_SMD:C_0603_1608Metric, symbol Device:C
- added J1: E+, TestPoint:TestPoint_Pad_2.0x2.0mm, symbol Connector_Generic:Conn_01x01
- added J2: A+, TestPoint:TestPoint_Pad_2.0x2.0mm, symbol Connector_Generic:Conn_01x01
- added J3: A-, TestPoint:TestPoint_Pad_2.0x2.0mm, symbol Connector_Generic:Conn_01x01
- added J4: E-, TestPoint:TestPoint_Pad_2.0x2.0mm, symbol Connector_Generic:Conn_01x01
- added J5: VBAT, TestPoint:TestPoint_Pad_2.0x2.0mm, symbol Connector_Generic:Conn_01x01
- added J6: GND, TestPoint:TestPoint_Pad_2.0x2.0mm, symbol Connector_Generic:Conn_01x01
- added Q1: Q_NMOS_GSD, Package_TO_SOT_SMD:SOT-23, symbol Transistor_FET:Q_NMOS_GSD
- added Q2: Q_PMOS_GSD, Package_TO_SOT_SMD:SOT-23, symbol Transistor_FET:Q_PMOS_GSD
- added R5, R6: 1k, Resistor_SMD:R_0402_1005Metric, symbol Device:R
- added R7, R8: 100k, Resistor_SMD:R_0402_1005Metric, symbol Device:R
- added U1: nrf52832_nRF52832, Package_DFN_QFN:Nordic_AQFN-73-1EP_7x7mm_P0.5mm, symbol nrf52832:nrf52832_nRF52832
- added U2: HX711, Package_SO:SOIC-16_3.9x9.9mm_P1.27mm, symbol Analog_ADC:HX711
- added U4: SHTC3, Sensor_Humidity:Sensirion_DFN-4-1EP_2x2mm_P1mm_EP0.7x1.6mm, symbol Sensor_Humidity:SHTC3
- added Y3: 32M, Ruuvi:20X16MM_4PIN_CRYSTAL, symbol Device:Crystal_GND24_Small
- C2: value 1u -> 1n; footprint RuuviTag:0402_CAP -> Capacitor_SMD:C_0402_1005Metric; now not fitted
- renumbered C15 to C1, C4 to C10, C10 to C11, C7 to C12, C5 to C13, C6 to C14, C11 to C16, C3 to C17, C13 to C18, C14 to C19, C19 to C20, C16 to C21, C1 to C22, C20 to C23, L4 to L1, L5 to L2, L1 to L3, L2 to L4, L3 to L5, P4 to P1, P15 to P10, P19 to P11, P20 to P12, P21 to P13, P8 to P15, P9 to P16, P18 to P17, P16 to P18, P5 to P19, P10 to P2, P23 to P20, P26 to P21, P17 to P22, P11 to P3, P22 to P4, P1 to P5, P24 to P6, P25 to P7, P13 to P8, P14 to P9, R3 to R1, R4 to R2, R1 to R3, R2 to R4
Connections:
- net GND: now also C15.2, C3.2, C4.2, C5.2, C7.2, J4.1 (Pin_1), J6.1 (Pin_1), Q1.2 (S), R8.2, U1.31 (VSS), U1.38 (P0.26), U1.45 (VSS), U1.49 (BOTPAD), U2.10 (INB+), U2.15 (RATE), U2.5 (AGND), U2.9 (INB-), U4.4 (VSS), Y3.2 (G), Y3.4 (G)
- net P0.20: now also U1.23 (P0.20/TRACECLK)
- net P0.30: now also U1.42 (P0.30/AIN6)
- net P0.31: now also U1.43 (P0.31/AIN7)
- net RESET: now also U1.24 (P0.21/RESET)
- net SCL: now also U1.7 (P0.05/AIN3), U4.3 (SDA)
- net SDA: now also U1.6 (P0.04/AIN2), U4.2 (SCL)
- net SENSOR_PWR_1: now also U1.15 (P0.12), U4.1 (VDD)
- net SWDCLK: now also U1.25 (SWDCLK)
- net SWDIO: now also U1.26 (SWDIO)
- net SWO: now also U1.21 (P0.18/TRACEDATA[0])
- net VDD: now also J5.1 (Pin_1), Q2.2 (S), R7.1, U1.13 (VDD), U1.36 (VDD), U1.48 (VDD)
- net XC1: now also U1.34 (XC1), Y3.1
- net XC2: now also U1.35 (XC2), Y3.3
- net ~{BUTTON}: now also U1.16 (P0.13)
- net ~{LED1}: now also U1.20 (P0.17)
- net ~{LED2}: now also U1.22 (P0.19)
- net at L4.1: now also U1.47 (DCDC)
- net at C16.2: now also C18.2, U1.1 (DEC1), U1.33 (DEC3)
- net at C14.2, L1.2: now also U1.11 (NFC1/P0.09)
- net at C12.1, L2.1: now also U1.12 (NFC2/P0.10)
- net at C10.2, Y1.1: now also U1.2 (P0.00/XL1)
- net at C13.2, Y1.2: now also U1.3 (P0.01/XL2)
- net at C22.1, L5.1: now also U1.30 (ANT)
- net at C17.1, L3.2: now also U1.46 (DEC4)
- net ANTENNA renamed ANT
- net SENSOR_PWR_2: no longer names the net of C2.1
- net SENSOR_PWR_2: now also C6.1, R5.1, U2.8 (INA+)
- net ~{TMP_ALERT}: no longer names the net of P21.7 (Pin_7)
- new net: Q1.3 (D), Q2.1 (G), R7.2
- new net: C4.1, C6.2, R6.2, U2.7 (INA-)
- new net: C7.1, U2.6 (VBG)
- new net HX711_DOUT: U1.10 (P0.08), U2.12 (DOUT)
- new net HX711_EN: Q1.1 (G), R8.1, U1.5 (P0.03/AIN1)
- new net HX711_PWR: C15.1, C3.1, C5.1, J1.1 (Pin_1), Q2.3 (D), U2.1 (VSUP), U2.16 (DVDD), U2.3 (AVDD), U2.4 (VFB)
- new net HX711_SCK: U1.9 (P0.07), U2.11 (PD_SCK)
- new net LC_A+: J2.1 (Pin_1), R5.2
- new net LC_A-: J3.1 (Pin_1), R6.1
- no-connect marks 9 -> 18
Other:
- note removed: "Accelerometer"
- note removed: "I2C Address: TMP116/7 = 0x48 (if ADDR = GND)"
- note removed: "Open-drain, requires a sw pull-up"
- note removed: "Pressure"
- note removed: "Temperature"
- moved on the sheet: C1, C11, C12, C14, C16, C18, C19, C20, C21, C22, C23, C8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

Commit message: chore: OpenWiki, Sensorboard-/ruuvitag_gas-Schaltplaene, Log-Level und Doku nachgezogen
- OpenWiki-Index (openwiki/, AGENTS.md) und Verweis in CLAUDE.md
- Sensorboard-Schaltplan/PCB und ruuvitag_gas-Schaltplan aktualisiert
- LDL1117S33R-Bauteilbibliothek, Material-Icon-Font 16 px
- display_config.h: Log-Level Main/Theme auf WARN, Screenshot-Block aufgeraeumt
- gasbee_nrf/README: HX711-Modul und AVDD-Spannungsteiler beschrieben
- ruuvitag_hw (Fremd-Repo) in .gitignore

Co-Authored-By: Claude Opus 5.5 <noreply@anthropic.com>
Other:
- note added: "Open-Source Gas Scale"
- note added: "RuuviTag_Gas"
- note removed: "Open-Source Sensor Beacon"
- note removed: "RuuviTag"
- note removed: "ruuvi.com"
- moved on the sheet: C1, C10, C11, C12, C13, C14, C15, C16, C17, C18, C19, C2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
